File: Wii-Nano Amp/Wii Custom Audio Board (I2S).kicad_pcb (KiCad board)
At the start: 2 copper layers, 37 x 39.3 mm, 28 parts, among them J1 SJ-3524-SMT, U1 LM49450SQ, U2 MCP1700T-2502E/TT

Commit message: Add files via upload
Parts:
- removed the CLK at (164.7, 75.9)
- removed I2S Audio: JST_XH_S4B-XH-A-1_1x04_P2.50mm_Horizontal, Connector_JST:JST_XH_S4B-XH-A-1_1x04_P2.50mm_Horizontal
- removed the MCLK at (164.2, 78.2)
- removed the SDI at (164.8, 73.2)
- removed the WS at (164.5, 70.8)
- added CLK: TestPoint_Pad_D1.5mm, TestPoint:TestPoint_Pad_D1.5mm, F.Cu at (158.7, 75.5)
- added MCLK: TestPoint_Pad_D1.5mm, TestPoint:TestPoint_Pad_D1.5mm, F.Cu at (158.7, 79.8)
- added SDI: TestPoint_Pad_D1.5mm, TestPoint:TestPoint_Pad_D1.5mm, F.Cu at (158.7, 71.2)
- added WS: TestPoint_Pad_D1.5mm, TestPoint:TestPoint_Pad_D1.5mm, F.Cu at (158.7, 66.8)
- moved +3V3 2.76 mm to (165.4, 90.7)
- moved GND 2.76 mm to (169.7, 90.7)
- moved SCL 0.43 mm to (158.7, 89.3)
- moved SDA 0.43 mm to (158.7, 85.0)
Routing:
- net Net-(U1-I2S_WS): track 18.5 -> 21.4 mm
- net Net-(U1-I2S_SDI): track 17.0 -> 18.2 mm
- net +3.3V: track 79.5 -> 78.5 mm
- net Net-(U1-SCL): track 17.2 -> 16.2 mm
- net Net-(U1-MCLK): track 13.7 -> 13.0 mm
Other:
- board text added: "Wii-Nano Amp Version: 1.4"
- board text removed: "Wii-Nano Amp Version: 1.3"
