File: Wii-Nano Power Delivery Board/Wii PD Board.kicad_sch (KiCad schematic)
At the start: 9 parts, among them J1 USB4105-GF-A, Q1 DMG3406L, U1 IP2721

Commit message: Add files via upload
Changed lines of the file:
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@@
 (kicad_sch (version 20230121) (generator eeschema)
   (paper "A4")
+  (junction (at 41.275 60.96) (diameter 0) (color 0 0 0 0)
+  )
   (junction (at 102.87 87.63) (diameter 0) (color 0 0 0 0)
   )
@@
   (junction (at 96.52 77.47) (diameter 0) (color 0 0 0 0)
   )
+  (junction (at 41.275 54.61) (diameter 0) (color 0 0 0 0)
+  )
   (junction (at 95.25 54.61) (diameter 0) (color 0 0 0 0)
   )
@@
   )
   (junction (at 96.52 80.01) (diameter 0) (color 0 0 0 0)
-  )
-  (junction (at 46.99 60.96) (diameter 0) (color 0 0 0 0)
-  )
-  (junction (at 46.99 54.61) (diameter 0) (color 0 0 0 0)
   )
   (junction (at 97.79 52.07) (diameter 0) (color 0 0 0 0)
@@
     (stroke (width 0) (type default))
   )
-  (wire (pts (xy 46.99 54.61) (xy 46.99 53.34))
+  (wire (pts (xy 41.275 54.61) (xy 41.275 53.34))
     (stroke (width 0) (type default))
   )
@@
     (stroke (width 0) (type default))
   )
-  (wire (pts (xy 46.99 55.88) (xy 46.99 54.61))
+  (wire (pts (xy 41.275 55.88) (xy 41.275 54.61))
     (stroke (width 0) (type default))
   )
@@
     (stroke (width 0) (type default))
   )
-  (wire (pts (xy 46.99 62.23) (xy 49.53 62.23))
+  (wire (pts (xy 41.275 62.23) (xy 49.53 62.23))
     (stroke (width 0) (type default))
   )
@@
     (stroke (width 0) (type default))
   )
-  (wire (pts (xy 46.99 59.69) (xy 49.53 59.69))
+  (wire (pts (xy 41.275 59.69) (xy 49.53 59.69))
     (stroke (width 0) (type default))
   )
@@
     (stroke (width 0) (type default))
   )
-  (wire (pts (xy 35.56 60.96) (xy 46.99 60.96))
+  (wire (pts (xy 35.56 60.96) (xy 41.275 60.96))
     (stroke (width 0) (type default))
   )
-  (wire (pts (xy 35.56 54.61) (xy 46.99 54.61))
+  (wire (pts (xy 35.56 54.61) (xy 41.275 54.61))
     (stroke (width 0) (type default))
   )
@@
     (stroke (width 0) (type default))
   )
-  (wire (pts (xy 46.99 60.96) (xy 46.99 59.69))
+  (wire (pts (xy 41.275 60.96) (xy 41.275 59.69))
     (stroke (width 0) (type default))
   )
@@
     (stroke (width 0) (type default))
   )
-  (wire (pts (xy 46.99 62.23) (xy 46.99 60.96))
+  (wire (pts (xy 41.275 62.23) (xy 41.275 60.96))
     (stroke (width 0) (type default))
   )
@@
     (stroke (width 0) (type default))
   )
-  (wire (pts (xy 46.99 53.34) (xy 49.53 53.34))
+  (wire (pts (xy 41.275 53.34) (xy 49.53 53.34))
     (stroke (width 0) (type default))
   )
-  (wire (pts (xy 49.53 55.88) (xy 46.99 55.88))
+  (wire (pts (xy 49.53 55.88) (xy 41.275 55.88))
     (stroke (width 0) (type default))
   )
